Commit message: nav2 work

File: ros2_packages/robot_nav/urdf/husky.urdf.xacro (robot description, xacro)
@@ -1,23 +1,23 @@
 <?xml version="1.0"?>
 <!--
-  Husky A200 URDF p/ simulação — mantém o chain base_footprint → base_link →
-  (wheels, base_laser) usado pelo slam_toolbox e Nav2.
+  Husky miniatura (URDF de apoio) — dimensões batem 1:1 com o husky.sdf
+  simulado no Gazebo. O robot_state_publisher usa esta árvore pra fornecer
+  os TFs estáticos que o slam_toolbox e o Nav2 consomem (principalmente
+  base_link → base_laser). O odom → base_link vem do plugin DiffDrive,
+  então base_link NÃO pode ter um outro pai aqui (sem base_footprint).
 -->
 <robot xmlns:xacro="http://www.ros.org/wiki/xacro" name="husky">
-  <xacro:property name="wheel_radius"  value="0.1651"/>
-  <xacro:property name="wheel_width"   value="0.1016"/>
-  <xacro:property name="track"         value="0.555"/>   <!-- separação esq-dir -->
-  <xacro:property name="wheelbase"     value="0.512"/>   <!-- dist frente-trás -->
-  <xacro:property name="body_length"   value="0.99"/>
-  <xacro:property name="body_width"    value="0.67"/>
-  <xacro:property name="body_height"   value="0.28"/>
-  <xacro:property name="lidar_x"       value="0.15"/>
-  <xacro:property name="lidar_z"       value="0.22"/>
-  <link name="base_footprint"/>
-  <joint name="base_footprint_joint" type="fixed">
-    <parent link="base_footprint"/>
-    <child link="base_link"/>
-    <origin xyz="0 0 ${wheel_radius}" rpy="0 0 0"/>
-  </joint>
+  <xacro:property name="wheel_radius"  value="0.06"/>
+  <xacro:property name="wheel_width"   value="0.03"/>
+  <xacro:property name="track"         value="0.24"/>   <!-- separação esq-dir -->
+  <xacro:property name="rear_wheel_x"  value="-0.09"/>  <!-- eixo traseiro -->
+  <xacro:property name="caster_x"      value="0.12"/>
+  <xacro:property name="caster_radius" value="0.03"/>
+  <xacro:property name="body_length"   value="0.31"/>
+  <xacro:property name="body_width"    value="0.24"/>
+  <xacro:property name="body_height"   value="0.14"/>
+  <!-- LiDAR centralizado em cima do corpo, coerente com husky.sdf -->
+  <xacro:property name="lidar_x"       value="0.0"/>
+  <xacro:property name="lidar_z"       value="0.09"/>
   <link name="base_link">
     <visual>
@@ -29,13 +29,13 @@
     </collision>
     <inertial>
-      <mass value="46.0"/>
-      <inertia ixx="0.6" ixy="0" ixz="0" iyy="1.8" iyz="0" izz="2.0"/>
+      <mass value="3.0"/>
+      <inertia ixx="0.025" ixy="0" ixz="0" iyy="0.035" iyz="0" izz="0.05"/>
     </inertial>
   </link>
-  <xacro:macro name="wheel" params="name x y roll">
+  <xacro:macro name="wheel" params="name x y">
     <joint name="${name}_joint" type="continuous">
       <parent link="base_link"/>
       <child link="${name}"/>
-      <origin xyz="${x} ${y} ${-body_height/2}" rpy="${roll} 0 0"/>
+      <origin xyz="${x} ${y} ${-body_height/2 + wheel_radius - wheel_radius}" rpy="${-pi/2} 0 0"/>
       <axis xyz="0 0 1"/>
     </joint>
@@ -49,25 +49,44 @@
       </collision>
       <inertial>
-        <mass value="2.5"/>
-        <inertia ixx="0.02" ixy="0" ixz="0" iyy="0.02" iyz="0" izz="0.03"/>
+        <mass value="0.2"/>
+        <inertia ixx="0.0003" ixy="0" ixz="0" iyy="0.0003" iyz="0" izz="0.0005"/>
       </inertial>
     </link>
   </xacro:macro>
-  <xacro:wheel name="front_left_wheel"  x="${ wheelbase/2}" y="${ track/2}" roll="${-pi/2}"/>
-  <xacro:wheel name="front_right_wheel" x="${ wheelbase/2}" y="${-track/2}" roll="${ pi/2}"/>
-  <xacro:wheel name="rear_left_wheel"   x="${-wheelbase/2}" y="${ track/2}" roll="${-pi/2}"/>
-  <xacro:wheel name="rear_right_wheel"  x="${-wheelbase/2}" y="${-track/2}" roll="${ pi/2}"/>
+  <xacro:wheel name="rear_left_wheel"   x="${rear_wheel_x}" y="${ track/2}"/>
+  <xacro:wheel name="rear_right_wheel"  x="${rear_wheel_x}" y="${-track/2}"/>
+  <!-- Roda boba (caster) — sphere fixa na frente, bate com o husky.sdf -->
+  <joint name="caster_joint" type="fixed">
+    <parent link="base_link"/>
+    <child link="caster_wheel"/>
+    <!-- z = -(wheel_radius + body_height/2 - caster_radius) p/ alinhar
+         com o chão quando base_link está em z=wheel_radius+body_height/2 -->
+    <origin xyz="${caster_x} 0 -0.10" rpy="0 0 0"/>
+  </joint>
+  <link name="caster_wheel">
+    <visual>
+      <geometry><sphere radius="${caster_radius}"/></geometry>
+      <material name="black"/>
+    </visual>
+    <collision>
+      <geometry><sphere radius="${caster_radius}"/></geometry>
+    </collision>
+    <inertial>
+      <mass value="0.05"/>
+      <inertia ixx="1e-5" ixy="0" ixz="0" iyy="1e-5" iyz="0" izz="1e-5"/>
+    </inertial>
+  </link>
   <joint name="laser_joint" type="fixed">
     <parent link="base_link"/>
     <child link="base_laser"/>
-    <origin xyz="${lidar_x} 0 ${body_height/2 + lidar_z - body_height/2}" rpy="0 0 0"/>
+    <origin xyz="${lidar_x} 0 ${lidar_z}" rpy="0 0 0"/>
   </joint>
   <link name="base_laser">
     <visual>
-      <geometry><cylinder radius="0.05" length="0.06"/></geometry>
+      <geometry><cylinder radius="0.038" length="0.04"/></geometry>
       <material name="blue"><color rgba="0.0 0.3 0.8 1.0"/></material>
     </visual>
     <collision>
-      <geometry><cylinder radius="0.05" length="0.06"/></geometry>
+      <geometry><cylinder radius="0.038" length="0.04"/></geometry>
     </collision>
     <inertial>

Commit message: RGB-D camera added

File: ros2_packages/robot_nav/urdf/husky.urdf.xacro (robot description, xacro)
@@ -95,3 +95,22 @@
     </inertial>
   </link>
+  <!-- Câmera RGB-D frontal — bate com a posição do <link name="camera_link">
+       no husky.sdf. URDF aqui só pra robot_state_publisher publicar o TF
+       estático base_link → camera_link, que o Nav2 e o map_service usam
+       pra transformar o point cloud e a imagem. -->
+  <joint name="camera_joint" type="fixed">
+    <parent link="base_link"/>
+    <child link="camera_link"/>
+    <origin xyz="0.16 0 0.02" rpy="0 0 0"/>
+  </joint>
+  <link name="camera_link">
+    <visual>
+      <geometry><box size="0.025 0.080 0.025"/></geometry>
+      <material name="black"><color rgba="0.1 0.1 0.1 1.0"/></material>
+    </visual>
+    <inertial>
+      <mass value="0.05"/>
+      <inertia ixx="0.00001" ixy="0" ixz="0" iyy="0.00001" iyz="0" izz="0.00001"/>
+    </inertial>
+  </link>
 </robot>

Commit message: Mais auditoria

File: ros2_packages/robot_nav/urdf/husky.urdf.xacro (robot description, xacro)
@@ -37,5 +37,5 @@
       <parent link="base_link"/>
       <child link="${name}"/>
-      <origin xyz="${x} ${y} ${-body_height/2 + wheel_radius - wheel_radius}" rpy="${-pi/2} 0 0"/>
+      <origin xyz="${x} ${y} ${-body_height/2}" rpy="${-pi/2} 0 0"/>
       <axis xyz="0 0 1"/>
     </joint>

File: ros2_packages/robot_nav/urdf/robot.urdf.xacro (robot description, xacro)
@@ -20,7 +20,10 @@
   <xacro:property name="lidar_x"          value="0.10"/>
   <xacro:property name="lidar_z"          value="0.12"/>
-  <!-- IMU (BNO055) e PMW3901 (optical flow) — montados no centro do chassi -->
+  <!-- IMU (BNO055) e PMW3901 (optical flow) — montados no centro do chassi.
+       flow_z é a altura do flow_link relativa ao base_link. Combinado com
+       base_link a wheel_radius=0.085 do chão, o sensor fica a 0.12 m do
+       chão — mesmo valor do default `flow_height` em trekking.launch.py. -->
   <xacro:property name="imu_z"            value="0.02"/>
-  <xacro:property name="flow_z"           value="-0.03"/>
+  <xacro:property name="flow_z"           value="0.035"/>
   <!-- ======= base_footprint ======= -->
   <link name="base_footprint"/>
@@ -47,5 +50,10 @@
     <inertial>
       <mass value="15.46"/>
-      <inertia ixx="0.5" ixy="0" ixz="0" iyy="0.5" iyz="0" izz="0.5"/>
+      <!-- Inércia da caixa 0.50×0.50×0.26 m para m=15.46 kg:
+             ixx = m(y²+z²)/12 ≈ 0.41
+             iyy = m(x²+z²)/12 ≈ 0.41
+             izz = m(x²+y²)/12 ≈ 0.64
+           Usado se algum dia migrarmos para sim com este URDF. -->
+      <inertia ixx="0.41" ixy="0" ixz="0" iyy="0.41" iyz="0" izz="0.64"/>
     </inertial>
   </link>
@@ -127,9 +135,9 @@
     </inertial>
   </link>
-  <!-- ======= Optical flow (PMW3901) — embaixo, olhando pro chão ======= -->
+  <!-- ======= Optical flow (PMW3901) — olhando pro chão ======= -->
   <joint name="flow_joint" type="fixed">
     <parent link="base_link"/>
     <child link="flow_link"/>
-    <origin xyz="0 0 ${-body_height/2 + flow_z}" rpy="0 ${pi} 0"/>
+    <origin xyz="0 0 ${flow_z}" rpy="0 ${pi} 0"/>
   </joint>
   <link name="flow_link">

Commit message: Aplica medios restantes da Etapa 3 da AUDITORIA_2026-05-18
- M1 odom_publisher: integracao com yaw no ponto medio do passo
- M2 sensors_imu: normaliza quaternion antes de enviar
- M3 mega_bridge: contador de frames descartados + warn throttled
- M5 Flow::read() retorna bool; txFlow checa retorno (simetrico ao txImu)
- M6 mega_bridge: bateria present via bit de fault (distingue 0V real de placa muda)
- M7 min_y_velocity_threshold 0.5 -> 0.001 (nav2_params{,_pi})
- M8 comentario distinguindo os dois xy_goal_tolerance
- M9 smoother min_velocity ree -0.15 -> -0.1 (alinha com DWB)
- M10 sim_robot.sdf: static_publisher false (evita duplicar TFs estaticos)
- M15 trekking_runner: stop zera current_idx
- M16 _led_tick: LED so publica quando a cor muda
- M18 comentario do camera_link (sensor removido, link/TF mantido)
- M20 comentario explicando controller_frequency 10 Hz

File: ros2_packages/robot_nav/urdf/husky.urdf.xacro (robot description, xacro)
@@ -95,8 +95,9 @@
     </inertial>
   </link>
-  <!-- Câmera RGB-D frontal — bate com a posição do <link name="camera_link">
-       no husky.sdf. URDF aqui só pra robot_state_publisher publicar o TF
-       estático base_link → camera_link, que o Nav2 e o map_service usam
-       pra transformar o point cloud e a imagem. -->
+  <!-- camera_link frontal — o SENSOR RGB-D foi removido do husky.sdf (M14):
+       não há mais bridge de /camera/*. Mantemos só o link visual + o TF
+       estático base_link → camera_link aqui pra um futuro upgrade de câmera
+       não precisar remexer geometria. Bate com o <link name="camera_link">
+       (visual) que continua no husky.sdf. -->
   <joint name="camera_joint" type="fixed">
     <parent link="base_link"/>
