Commit message: New chassi automation + arduino mega + sensors + ligth

File: ros2_packages/robot_nav/urdf/robot.urdf.xacro (robot description, xacro)
@@ -1,23 +1,27 @@
 <?xml version="1.0"?>
-<robot xmlns:xacro="http://www.ros.org/wiki/xacro" name="hoverboard_robot">
+<robot xmlns:xacro="http://www.ros.org/wiki/xacro" name="robo_4_rodas">
   <!-- ============================================================
-       Hoverboard Robot Description
-       Adjust dimensions to match your actual robot:
-         wheel_radius: radius of the hoverboard wheels (meters)
-         wheel_base:   distance between left and right wheel centers (meters)
-         lidar_x:      lidar forward offset from robot center (meters)
-         lidar_z:      lidar height above base_link (meters)
+       Robô skid-steer 4 rodas (2 placas de hoverboard, ponte MEGA).
+       Dimensões medidas no chassi atual (2026-05-11):
+         carcaça externa : 50 × 50 × 26 cm
+         estrutura interna: 37 × 35 × 16 cm (alumínio)
+         roda hoverboard : raio 8,5 cm  largura 6 cm
+         bitola (esq-dir): 50 cm
+         entre-eixos     : 37 cm
        ============================================================ -->
-  <xacro:property name="wheel_radius" value="0.085"/>
-  <xacro:property name="wheel_width"  value="0.06"/>
-  <xacro:property name="wheel_base"   value="0.45"/>
-  <xacro:property name="body_length"  value="0.50"/>
-  <xacro:property name="body_width"   value="0.45"/>
-  <xacro:property name="body_height"  value="0.10"/>
-  <!-- LiDAR position: slightly forward and on top -->
-  <xacro:property name="lidar_x"      value="0.10"/>
-  <xacro:property name="lidar_z"      value="0.12"/>
-  <!-- pi já existe no xacro como constante embutida -->
-  <!-- ======= base_footprint (ground projection) ======= -->
+  <xacro:property name="wheel_radius"     value="0.085"/>
+  <xacro:property name="wheel_width"      value="0.06"/>
+  <xacro:property name="track_width"      value="0.50"/>   <!-- bitola: distância entre centros L-R -->
+  <xacro:property name="wheelbase"        value="0.37"/>   <!-- entre-eixos: distância entre eixos F-R -->
+  <xacro:property name="body_length"      value="0.50"/>
+  <xacro:property name="body_width"       value="0.50"/>
+  <xacro:property name="body_height"      value="0.26"/>
+  <!-- LiDAR no topo, ligeiramente à frente -->
+  <xacro:property name="lidar_x"          value="0.10"/>
+  <xacro:property name="lidar_z"          value="0.12"/>
+  <!-- IMU (BNO055) e PMW3901 (optical flow) — montados no centro do chassi -->
+  <xacro:property name="imu_z"            value="0.02"/>
+  <xacro:property name="flow_z"           value="-0.03"/>
+  <!-- ======= base_footprint ======= -->
   <link name="base_footprint"/>
   <joint name="base_footprint_joint" type="fixed">
@@ -26,5 +30,5 @@
     <origin xyz="0 0 ${wheel_radius}" rpy="0 0 0"/>
   </joint>
-  <!-- ======= base_link (center of robot body) ======= -->
+  <!-- ======= base_link ======= -->
   <link name="base_link">
     <visual>
@@ -42,60 +46,40 @@
     </collision>
     <inertial>
-      <mass value="10.0"/>
-      <inertia ixx="0.1" ixy="0" ixz="0" iyy="0.1" iyz="0" izz="0.1"/>
+      <mass value="15.46"/>
+      <inertia ixx="0.5" ixy="0" ixz="0" iyy="0.5" iyz="0" izz="0.5"/>
     </inertial>
   </link>
-  <!-- ======= Left Wheel ======= -->
-  <joint name="left_wheel_joint" type="continuous">
-    <parent link="base_link"/>
-    <child link="left_wheel"/>
-    <origin xyz="0 ${wheel_base/2} ${-body_height/2}" rpy="${-pi/2} 0 0"/>
-    <axis xyz="0 0 1"/>
-  </joint>
-  <link name="left_wheel">
-    <visual>
-      <geometry>
-        <cylinder radius="${wheel_radius}" length="${wheel_width}"/>
-      </geometry>
-      <material name="black">
-        <color rgba="0.1 0.1 0.1 1.0"/>
-      </material>
-    </visual>
-    <collision>
-      <geometry>
-        <cylinder radius="${wheel_radius}" length="${wheel_width}"/>
-      </geometry>
-    </collision>
-    <inertial>
-      <mass value="1.5"/>
-      <inertia ixx="0.005" ixy="0" ixz="0" iyy="0.005" iyz="0" izz="0.009"/>
-    </inertial>
-  </link>
-  <!-- ======= Right Wheel ======= -->
-  <joint name="right_wheel_joint" type="continuous">
-    <parent link="base_link"/>
-    <child link="right_wheel"/>
-    <origin xyz="0 ${-wheel_base/2} ${-body_height/2}" rpy="${pi/2} 0 0"/>
-    <axis xyz="0 0 1"/>
-  </joint>
-  <link name="right_wheel">
-    <visual>
-      <geometry>
-        <cylinder radius="${wheel_radius}" length="${wheel_width}"/>
-      </geometry>
-      <material name="black">
-        <color rgba="0.1 0.1 0.1 1.0"/>
-      </material>
-    </visual>
-    <collision>
-      <geometry>
-        <cylinder radius="${wheel_radius}" length="${wheel_width}"/>
-      </geometry>
-    </collision>
-    <inertial>
-      <mass value="1.5"/>
-      <inertia ixx="0.005" ixy="0" ixz="0" iyy="0.005" iyz="0" izz="0.009"/>
-    </inertial>
-  </link>
+  <!-- ======= Macro de roda ======= -->
+  <xacro:macro name="wheel" params="name x y">
+    <joint name="${name}_joint" type="continuous">
+      <parent link="base_link"/>
+      <child link="${name}"/>
+      <origin xyz="${x} ${y} ${-body_height/2}" rpy="${-pi/2} 0 0"/>
+      <axis xyz="0 0 1"/>
+    </joint>
+    <link name="${name}">
+      <visual>
+        <geometry>
+          <cylinder radius="${wheel_radius}" length="${wheel_width}"/>
+        </geometry>
+        <material name="black">
+          <color rgba="0.1 0.1 0.1 1.0"/>
+        </material>
+      </visual>
+      <collision>
+        <geometry>
+          <cylinder radius="${wheel_radius}" length="${wheel_width}"/>
+        </geometry>
+      </collision>
+      <inertial>
+        <mass value="1.5"/>
+        <inertia ixx="0.005" ixy="0" ixz="0" iyy="0.005" iyz="0" izz="0.009"/>
+      </inertial>
+    </link>
+  </xacro:macro>
+  <xacro:wheel name="front_left_wheel"  x="${ wheelbase/2}" y="${ track_width/2}"/>
+  <xacro:wheel name="front_right_wheel" x="${ wheelbase/2}" y="${-track_width/2}"/>
+  <xacro:wheel name="rear_left_wheel"   x="${-wheelbase/2}" y="${ track_width/2}"/>
+  <xacro:wheel name="rear_right_wheel"  x="${-wheelbase/2}" y="${-track_width/2}"/>
   <!-- ======= LiDAR (FHL-LD20) ======= -->
   <joint name="laser_joint" type="fixed">
@@ -123,3 +107,43 @@
     </inertial>
   </link>
+  <!-- ======= IMU (BNO055) ======= -->
+  <joint name="imu_joint" type="fixed">
+    <parent link="base_link"/>
+    <child link="imu_link"/>
+    <origin xyz="0 0 ${imu_z}" rpy="0 0 0"/>
+  </joint>
+  <link name="imu_link">
+    <visual>
+      <geometry>
+        <box size="0.02 0.02 0.005"/>
+      </geometry>
+      <material name="red">
+        <color rgba="0.8 0.1 0.1 1.0"/>
+      </material>
+    </visual>
+    <inertial>
+      <mass value="0.01"/>
+      <inertia ixx="1e-5" ixy="0" ixz="0" iyy="1e-5" iyz="0" izz="1e-5"/>
+    </inertial>
+  </link>
+  <!-- ======= Optical flow (PMW3901) — embaixo, olhando pro chão ======= -->
+  <joint name="flow_joint" type="fixed">
+    <parent link="base_link"/>
+    <child link="flow_link"/>
+    <origin xyz="0 0 ${-body_height/2 + flow_z}" rpy="0 ${pi} 0"/>
+  </joint>
+  <link name="flow_link">
+    <visual>
+      <geometry>
+        <box size="0.02 0.02 0.005"/>
+      </geometry>
+      <material name="green">
+        <color rgba="0.1 0.7 0.1 1.0"/>
+      </material>
+    </visual>
+    <inertial>
+      <mass value="0.01"/>
+      <inertia ixx="1e-5" ixy="0" ixz="0" iyy="1e-5" iyz="0" izz="1e-5"/>
+    </inertial>
+  </link>
 </robot>

Commit message: Aplica Etapas 1+2 da AUDITORIA_2026-05-18
Críticos:
- C1 URDF: base_footprint_joint em wheel_radius+body_height/2 (REP-103);
  flow_z ajustado pra manter sensor a 0.12 m do chão
- C2 trekking_runner: _state_lock + snapshot em pose/cones/control/state
- C3 mega_bridge: RX thread enfileira em queue; timer 200 Hz publica dentro do executor
- C4 app: _TREKKING_CMDS alinhado com _on_cmd do runner (clear adicionado,
  start/remove_last/index removidos)

Altos:
- A1 /light/marker (Bool) com estado relé+marker preservado entre callbacks
- A2 firmware preenche faultF/faultR + sensor_flags; bridge publica /system/health (JSON)
- A3 pose_estimator: warn throttled e /trekking/health (JSON) quando flow stale/alpha baixo
- A4 map_service: lock em load_route e no _wp_active=False final do runner
- A5 _on_cmd load_waypoints: try/except por waypoint malformado
- A6 _on_button: debounce de 2 frames consecutivos antes do rising edge
- A7 Flow::read: recovery automático a cada 2 s (mesmo padrão do Imu)
- A8 nav2_params{,_pi}.yaml: min_obstacle_height 0.0 (LiDAR-only)
- A9 comentários ~/ros2_ws → install/setup.bash (app.py, robot_controller.py)
- A10 broadcast=False → room=request.sid em key_event/gamepad_event

File: ros2_packages/robot_nav/urdf/robot.urdf.xacro (robot description, xacro)
@@ -21,15 +21,19 @@
   <xacro:property name="lidar_z"          value="0.12"/>
   <!-- IMU (BNO055) e PMW3901 (optical flow) — montados no centro do chassi.
-       flow_z é a altura do flow_link relativa ao base_link. Combinado com
-       base_link a wheel_radius=0.085 do chão, o sensor fica a 0.12 m do
-       chão — mesmo valor do default `flow_height` em trekking.launch.py. -->
+       flow_z é o offset do flow_link em relação ao base_link (CoM do corpo).
+       Combinado com base_link a (wheel_radius + body_height/2) = 0.215 m do
+       chão, e flow_z = -0.095, o sensor fica a 0.12 m do chão — mesmo valor
+       do default `flow_height` em trekking.launch.py. -->
   <xacro:property name="imu_z"            value="0.02"/>
-  <xacro:property name="flow_z"           value="0.035"/>
+  <xacro:property name="flow_z"           value="-0.095"/>
   <!-- ======= base_footprint ======= -->
   <link name="base_footprint"/>
+  <!-- base_link no CoM do corpo (REP-103). Posição do chão:
+       wheel_radius (centro da roda) + body_height/2 (do centro da roda ao
+       CoM do corpo, já que o eixo da roda está alinhado ao fundo do corpo). -->
   <joint name="base_footprint_joint" type="fixed">
     <parent link="base_footprint"/>
     <child link="base_link"/>
-    <origin xyz="0 0 ${wheel_radius}" rpy="0 0 0"/>
+    <origin xyz="0 0 ${wheel_radius + body_height/2}" rpy="0 0 0"/>
   </joint>
   <!-- ======= base_link ======= -->

Commit message: fix(robot): LiDAR no CENTRO — remove offset x falso de 0.10m (URDF + cone_detector)
Todos os sensores ficam no centro do robô. O lidar_x=0.10 do URDF virava
o TF base_link->base_laser: SLAM e costmaps achavam que o scan nascia
10cm à frente do real (obstáculos frontais 10cm 'mais longe' no costmap,
traseiros 10cm 'mais perto'). cone_detector/trekking idem nos cones.
ATENÇÃO: o mapa golden foi construído com o TF antigo — validar
localização nele na próxima sessão com robô.

File: ros2_packages/robot_nav/urdf/robot.urdf.xacro (robot description, xacro)
@@ -17,6 +17,9 @@
   <xacro:property name="body_width"       value="0.50"/>
   <xacro:property name="body_height"      value="0.26"/>
-  <!-- LiDAR no topo, ligeiramente à frente -->
-  <xacro:property name="lidar_x"          value="0.10"/>
+  <!-- LiDAR no topo, no CENTRO do robô (2026-06-11: o 0.10 antigo era falso;
+       TODOS os sensores são centrais). Este valor vira o TF
+       base_link→base_laser usado por SLAM/costmaps — com 0.10, todo scan
+       nascia 10cm à frente do real. -->
+  <xacro:property name="lidar_x"          value="0.0"/>
   <xacro:property name="lidar_z"          value="0.12"/>
   <!-- IMU (BNO055) e PMW3901 (optical flow) — montados no centro do chassi.
