Commit message: feat(imu): BNO055 como segunda IMU (9 eixos + heading absoluto)
A BNO055 entra AO LADO da MPU, no mesmo I²C da MEGA (0x28/0x29 contra
0x68), como terceira fonte de giro e direção. Dois caminhos independentes,
os dois desligáveis por parâmetro de launch:

  - taxa de yaw: média ponderada com o gyro da MPU (imu2_rate_weight=0.5)
  - heading ABSOLUTO: o quaternion NDOF ancora o yaw no norte magnético e
    tira a deriva do yaw integrado — o ganho principal no trekking, onde o
    percurso é longo e não há LiDAR reancorando a pose.

A correção de heading é lenta (heading_gain=0.2, τ≈5 s) e saturada
(heading_max_rate=0.15 rad/s): nunca "yaw = yaw do mag", porque um ímã no
chão viraria salto de heading e no Nav2 salto de heading vira manobra real
do robô. O alinhamento norte↔odom é latcheado na 1ª amostra aceita, então a
correção nasce valendo zero e só combate deriva; o yaw_fix da web arrasta
esse offset junto, então correção manual não é desfeita pela âncora.

Guardas contra os dois modos de falha silenciosa:
  - gate de discordância: se as duas IMUs lerem giro real com sinais opostos
    (BNO055 montada girada), a média daria ZERO — robô gira no chão sem
    girar no mapa. A #2 é descartada no tick e o nó loga error apontando
    imu2_yaw_sign.
  - gate de calibração: heading só é usado com o campo mag de /imu2/calib
    >= 2; mag descalibrado ainda entrega quaternion, apontando pra um norte
    inventado.

A BNO055 NÃO entra na translação: integrar accel duas vezes diverge em
metros por minuto. O ganho dela na posição é indireto e maior — a direção
pra onde a velocidade de roda/flow é projetada deixa de derivar.

Firmware: driver próprio sensors_bno055.* (registrador direto, sem Adafruit,
pra respeitar o Wire.setWireTimeout() anti-hang), frame FT_IMU2 (0x85, 27
bytes) a 50 Hz defasado 10 ms do FT_IMU, bit 2 de sensor_flags. O reset por
software da BNO055 bloqueia ~700 ms e só acontece no BOOT: em runtime
estouraria o SETPOINT_TIMEOUT_MS (500 ms) do hoverboard e o robô daria um
solavanco a cada tentativa de recovery.

Sensor OPCIONAL: sem a BNO055 montada tudo roda como antes, sem warn.
use_imu2:=false corta os dois caminhos; use_imu2_heading:=false desliga só
a âncora (para ambiente com muito ferro/EMI).

Validado só em software (o sensor ainda não está montado): 303 testes do
robot_nav passam, 10 deles novos no núcleo puro; smoke test do nó real com
BNO055 sintética mostrou a âncora derrubando 20 s de bias de 0.02 rad/s de
+22.9° para +5.6°, yaw_fix sobrevivendo e o gate de sinal mantendo o giro em
+45.9° em vez de zerar. Firmware compila limpo: RAM 12.8%, flash 5.8%.
Passos de bancada com o sensor na mão: CONEXOES.txt e ESTADO_PROJETO.md.

Co-Authored-By: Claude Opus 5 <noreply@anthropic.com>
Claude-Session: https://claude.ai/code/session_01NjPB5tJHxr32suNxvfkDUa

File: ros2_packages/robot_nav/urdf/robot.urdf.xacro (robot description, xacro)
@@ -23,5 +23,5 @@
   <xacro:property name="lidar_x"          value="0.0"/>
   <xacro:property name="lidar_z"          value="0.12"/>
-  <!-- IMU (BNO055) e PMW3901 (optical flow) — montados no centro do chassi.
+  <!-- IMUs (MPU6050 + BNO055) e PMW3901 (optical flow) — no centro do chassi.
        flow_z é o offset do flow_link em relação ao base_link (CoM do corpo).
        Combinado com base_link a (wheel_radius + body_height/2) = 0.215 m do
@@ -122,5 +122,5 @@
     </inertial>
   </link>
-  <!-- ======= IMU (BNO055) ======= -->
+  <!-- ======= IMU #1 (MPU6050 — gyro/accel, sem mag) ======= -->
   <joint name="imu_joint" type="fixed">
     <parent link="base_link"/>
@@ -135,4 +135,31 @@
       <material name="red">
         <color rgba="0.8 0.1 0.1 1.0"/>
+      </material>
+    </visual>
+    <inertial>
+      <mass value="0.01"/>
+      <inertia ixx="1e-5" ixy="0" ixz="0" iyy="1e-5" iyz="0" izz="1e-5"/>
+    </inertial>
+  </link>
+  <!-- ======= IMU #2 (BNO055 — 9 eixos, heading absoluto) =======
+       Ao LADO da #1, no mesmo I²C da MEGA. O deslocamento em x/y é irrelevante
+       pro que consumimos dela (giro e orientação não dependem de onde o sensor
+       está no corpo rígido); o link existe pro frame_id de /imu2/data e
+       /imu2/mag resolver no TF e pro RViz mostrar onde a peça está.
+       ATENÇÃO: se a BNO055 for montada GIRADA em relação ao chassi, o lugar de
+       corrigir NÃO é o rpy daqui — é o `imu2_yaw_sign` do pose_estimator (o nó
+       lê os dados no frame BRUTO do sensor, sem passar pelo TF). -->
+  <joint name="imu2_joint" type="fixed">
+    <parent link="base_link"/>
+    <child link="imu2_link"/>
+    <origin xyz="0.03 0 ${imu_z}" rpy="0 0 0"/>
+  </joint>
+  <link name="imu2_link">
+    <visual>
+      <geometry>
+        <box size="0.02 0.02 0.005"/>
+      </geometry>
+      <material name="orange">
+        <color rgba="0.9 0.5 0.1 1.0"/>
       </material>
     </visual>
