Commit message: sim: corrige geometria — chassi 0.37×0.35 (não 0.50×0.50) e LiDAR no topo
Feedback em campo: eu tinha posto o corpo como 0.50×0.50 (a carcaça
EXTERNA), mas o chassi real é 0.37 (frente-trás) × 0.35 (esq-dir). O
0.50×0.50 é o vão RODA-A-RODA, que as rodas (track 0.50) já fazem — o
chassi fica por dentro. E o LiDAR estava flutuando 0.12m acima do corpo
(robô real não tem mastro) -> assentado no topo do chassi (z 0.25->0.15).
Inércia recalculada p/ a caixa 0.37×0.35×0.26. Revalidado no gz Harmonic
(spawn/reto/giro/lidar OK).

File: ros2_packages/robot_nav/urdf/sim_robot.urdf.xacro (robot description, xacro)
@@ -17,11 +17,13 @@
   <xacro:property name="track_width"   value="0.50"/>   <!-- bitola esq-dir -->
   <xacro:property name="wheelbase"     value="0.37"/>   <!-- entre-eixos F-R -->
-  <xacro:property name="body_length"   value="0.50"/>
-  <xacro:property name="body_width"    value="0.50"/>
+  <!-- Chassi (estrutura interna): 0.37 frente-trás × 0.35 esq-dir. O footprint
+       roda-a-roda ~0.50×0.50 vem das RODAS (track 0.50), o chassi fica por dentro. -->
+  <xacro:property name="body_length"   value="0.37"/>
+  <xacro:property name="body_width"    value="0.35"/>
   <xacro:property name="body_height"   value="0.26"/>
-  <!-- LiDAR no CENTRO (2026-06-11: o 0.10 antigo era falso). Offset em z bate
-       com o real: body_height/2 + lidar_z = 0.13 + 0.12 = 0.25 acima do base_link. -->
+  <!-- LiDAR no CENTRO (2026-06-11: o 0.10 antigo era falso), assentado no TOPO
+       do chassi (sem mastro): z = body_height/2 + lidar_z = 0.13 + 0.02 = 0.15. -->
   <xacro:property name="lidar_x"       value="0.0"/>
-  <xacro:property name="lidar_z"       value="0.12"/>
+  <xacro:property name="lidar_z"       value="0.02"/>
   <link name="base_link">
     <visual>
@@ -34,5 +36,5 @@
     <inertial>
       <mass value="15.46"/>
-      <inertia ixx="0.41" ixy="0" ixz="0" iyy="0.41" iyz="0" izz="0.64"/>
+      <inertia ixx="0.25" ixy="0" ixz="0" iyy="0.26" iyz="0" izz="0.33"/>
     </inertial>
   </link>

Commit message: sim: geometria real do chassi + eixo/mancal (rodas nao flutuam mais)
Medidas confirmadas: ponta-a-ponta das rodas = 0.50 nas 2 direcoes -> track
0.44 (0.50-largura 0.06), wheelbase 0.33 (0.50-diametro 0.17); chassi
0.37x0.35x0.16 (altura era 0.26). LiDAR no topo (z=0.10). Eixo+mancal ligando
roda ao chassi (antes pareciam flutuar; na fisica sempre tocaram o chao).
Validado gz: corpo assenta z=0.165 e TRANSLADA (x 0->0.97 c/ cmd_vel direto).
O 'nao se mexe' NAO e o modelo, e o caminho teleop->cmd_vel.

File: ros2_packages/robot_nav/urdf/sim_robot.urdf.xacro (robot description, xacro)
@@ -12,14 +12,16 @@
 -->
 <robot xmlns:xacro="http://www.ros.org/wiki/xacro" name="sim_robot">
-  <!-- Dimensões medidas no chassi real (2026-05-11) — iguais ao robot.urdf.xacro -->
+  <!-- Medidas reais do chassi (2026-06-24, confirmadas). Ponta-a-ponta das
+       rodas = 0.50 nas DUAS direções -> centros: track = 0.50-wheel_width(0.06)
+       = 0.44; wheelbase = 0.50-diâmetro(0.17) = 0.33. -->
   <xacro:property name="wheel_radius"  value="0.085"/>
   <xacro:property name="wheel_width"   value="0.06"/>
-  <xacro:property name="track_width"   value="0.50"/>   <!-- bitola esq-dir -->
-  <xacro:property name="wheelbase"     value="0.37"/>   <!-- entre-eixos F-R -->
-  <!-- Chassi (estrutura interna): 0.37 frente-trás × 0.35 esq-dir. O footprint
-       roda-a-roda ~0.50×0.50 vem das RODAS (track 0.50), o chassi fica por dentro. -->
+  <xacro:property name="track_width"   value="0.44"/>   <!-- centros esq-dir -->
+  <xacro:property name="wheelbase"     value="0.33"/>   <!-- centros F-R -->
+  <!-- Chassi: 0.37 frente-trás × 0.35 esq-dir × 0.16 altura. As rodas ficam
+       POR FORA (ponta-a-ponta 0.50×0.50), conectadas por eixo no chassi. -->
   <xacro:property name="body_length"   value="0.37"/>
   <xacro:property name="body_width"    value="0.35"/>
-  <xacro:property name="body_height"   value="0.26"/>
+  <xacro:property name="body_height"   value="0.16"/>
   <!-- LiDAR no CENTRO (2026-06-11: o 0.10 antigo era falso), assentado no TOPO
        do chassi (sem mastro): z = body_height/2 + lidar_z = 0.13 + 0.02 = 0.15. -->
@@ -36,5 +38,5 @@
     <inertial>
       <mass value="15.46"/>
-      <inertia ixx="0.25" ixy="0" ixz="0" iyy="0.26" iyz="0" izz="0.33"/>
+      <inertia ixx="0.19" ixy="0" ixz="0" iyy="0.21" iyz="0" izz="0.33"/>
     </inertial>
   </link>

Commit message: sim: corrige GIRO (fdir1+mu2) e geometria eixo/mancal
Giro nao funcionava (38% do comandado + derrapa 0.49m). Fix: fdir1=(1 0 0) direcao de rolagem, mu 1.2 (grip), mu2 0.1 (lateral escorrega) -> gira no lugar (drift 4cm), sentido certo. Geometria: mancal 3.5cm topo no chassi + eixo no meio -> base_link z=0.1825, rodas z_rel -0.0975 (tocam chao), eixo curto 0.05 (era 0.20), roda por fora do mancal. URDF acompanha. Validado gz: reto x 0->1.0, giro no lugar.

File: ros2_packages/robot_nav/urdf/sim_robot.urdf.xacro (robot description, xacro)
@@ -41,4 +41,7 @@
     </inertial>
   </link>
+  <!-- Mancal de 3.5cm entre o fundo do chassi e o eixo: a roda fica 0.0175
+       (meio mancal) abaixo do fundo do chassi. Bate com o sim_robot.sdf. -->
+  <xacro:property name="mancal_h" value="0.035"/>
   <!-- Macro de roda — eixo de giro alinhado a Y (rpy -pi/2 em X), igual ao real -->
   <xacro:macro name="wheel" params="name x y">
@@ -46,5 +49,5 @@
       <parent link="base_link"/>
       <child link="${name}"/>
-      <origin xyz="${x} ${y} ${-body_height/2}" rpy="${-pi/2} 0 0"/>
+      <origin xyz="${x} ${y} ${-(body_height/2 + mancal_h/2)}" rpy="${-pi/2} 0 0"/>
       <axis xyz="0 0 1"/>
     </joint>
